File: Esq_Eagle/Luva/LuvaAcel.brd (EAGLE design)
At the start: 39 x 52.5 mm, 7 parts, among them U1 GY-521MPU6050

Commit message: gerando arquivo para impressao das placas
Parts:
- removed U$1: PRO-MINI-2, Arduino-clone:PRO-MINI-2
- added A4ARD, A5ARD, GNDARD, RXARD, TXARD, VCCARD: (no value), wirepad:3,17/1,1
- moved U1 17.9 mm to (34.8, 20.6)
- moved U$2 1.41 mm to (-12.1, 25.3)
Connections:
- net N$1: now also A5ARD.1; no longer U$1.A5
- net N$2: now also A4ARD.1; no longer U$1.A4
- net N$4: now also GNDARD.1; no longer U$1.GND
- net N$5: now also TXARD.1; no longer U$1.TX0
- net N$6: now also RXARD.1; no longer U$1.RX1
- net N$7: now also VCCARD.1; no longer U$1.RAW, U$2.6
Routing:
- net N$1: track 64.5 -> 9.36 mm
- net N$2: track 50.9 -> 10.3 mm
- net N$5: track 46.0 -> 8.38 mm
- net N$6: track 22.3 -> 7.50 mm
- net N$7: track 72.8 -> 60.1 mm
- net N$4: track 66.3 -> 70.3 mm
Other:
- board size 39 x 52.5 mm -> 33 x 35.5 mm
