File: Esq_Eagle/Luva/LuvaAcel.sch (EAGLE design)
At the start: 7 parts, among them U1 GY-521MPU6050

Commit message: gerando arquivo para impressao das placas
Parts:
- removed U$1: PRO-MINI-2, Arduino-clone:PRO-MINI-2
- added A4ARD, A5ARD, GNDARD, RXARD, TXARD, VCCARD: (no value), wirepad:3,17/1,1
Connections:
- net N$1: now also A5ARD.P; no longer U$1.A5
- net N$2: now also A4ARD.P; no longer U$1.A4
- net N$4: now also GNDARD.P; no longer U$1.GND
- net N$5: now also TXARD.P; no longer U$1.TX0
- net N$6: now also RXARD.P; no longer U$1.RX1
- net N$7: now also VCCARD.P; no longer U$1.RAW, U$2.EN
Other:
- moved on the sheet: VCC
Changed lines of the file:
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@@
 <?xml version="1.0" encoding="utf-8"?>
 <!DOCTYPE eagle SYSTEM "eagle.dtd">
-<eagle version="9.5.1">
+<eagle version="6.6.0">
 <drawing>
 <settings>
@@
 </classes>
 <parts>
-<part name="U$1" library="Arduino-clone" deviceset="PRO-MINI-2" device=""/>
 <part name="U1" library="gy-521" deviceset="GY-521" device="MPU6050"/>
-<part name="VCC" library="wirepad" library_urn="urn:adsk.eagle:library:412" deviceset="3,17/1,1" device="" package3d_urn="urn:adsk.eagle:package:30832/1"/>
-<part name="GND" library="wirepad" library_urn="urn:adsk.eagle:library:412" deviceset="3,17/1,1" device="" package3d_urn="urn:adsk.eagle:package:30832/1"/>
+<part name="VCC" library="wirepad" deviceset="3,17/1,1" device=""/>
+<part name="GND" library="wirepad" deviceset="3,17/1,1" device=""/>
 <part name="U$2" library="diy-modules" deviceset="WIRELESS-BLUETOOTH-HC-05" device=""/>
-<part name="INTER1" library="wirepad" library_urn="urn:adsk.eagle:library:412" deviceset="3,17/1,1" device="" package3d_urn="urn:adsk.eagle:package:30832/1"/>
-<part name="INTER2" library="wirepad" library_urn="urn:adsk.eagle:library:412" deviceset="3,17/1,1" device="" package3d_urn="urn:adsk.eagle:package:30832/1"/>
+<part name="INTER1" library="wirepad" deviceset="3,17/1,1" device=""/>
+<part name="INTER2" library="wirepad" deviceset="3,17/1,1" device=""/>
+<part name="GNDARD" library="wirepad" deviceset="3,17/1,1" device=""/>
+<part name="VCCARD" library="wirepad" deviceset="3,17/1,1" device=""/>
+<part name="A4ARD" library="wirepad" deviceset="3,17/1,1" device=""/>
+<part name="A5ARD" library="wirepad" deviceset="3,17/1,1" device=""/>
+<part name="RXARD" library="wirepad" deviceset="3,17/1,1" device=""/>
+<part name="TXARD" library="wirepad" deviceset="3,17/1,1" device=""/>
 </parts>
 <sheets>
@@
 </plain>
 <instances>
-<instance part="U$1" gate="G$1" x="50.8" y="40.64" smashed="yes" rot="R90"/>
 <instance part="U1" gate="G$1" x="114.3" y="45.72" smashed="yes"/>
-<instance part="VCC" gate="1" x="43.18" y="78.74" smashed="yes">
-<attribute name="NAME" x="42.037" y="80.5942" size="1.778" layer="95"/>
-<attribute name="VALUE" x="42.037" y="75.438" size="1.778" layer="96"/>
+<instance part="VCC" gate="1" x="45.72" y="78.74" smashed="yes">
+<attribute name="NAME" x="44.577" y="80.5942" size="1.778" layer="95"/>
+<attribute name="VALUE" x="44.577" y="75.438" size="1.778" layer="96"/>
 </instance>
 <instance part="GND" gate="1" x="43.18" y="71.12" smashed="yes">
@@
 <attribute name="NAME" x="67.8942" y="82.423" size="1.778" layer="95" rot="R270"/>
 <attribute name="VALUE" x="62.738" y="82.423" size="1.778" layer="96" rot="R270"/>
+</instance>
+<instance part="GNDARD" gate="1" x="40.64" y="43.18" smashed="yes" rot="R90">
+<attribute name="NAME" x="38.7858" y="42.037" size="1.778" layer="95" rot="R90"/>
+<attribute name="VALUE" x="43.942" y="42.037" size="1.778" layer="96" rot="R90"/>
+</instance>
+<instance part="VCCARD" gate="1" x="20.32" y="78.74" smashed="yes">
+<attribute name="NAME" x="19.177" y="80.5942" size="1.778" layer="95"/>
+<attribute name="VALUE" x="19.177" y="75.438" size="1.778" layer="96"/>
+</instance>
+<instance part="A4ARD" gate="1" x="81.28" y="45.72" smashed="yes">
+<attribute name="NAME" x="80.137" y="47.5742" size="1.778" layer="95"/>
+<attribute name="VALUE" x="80.137" y="42.418" size="1.778" layer="96"/>
+</instance>
+<instance part="A5ARD" gate="1" x="81.28" y="50.8" smashed="yes">
+<attribute name="NAME" x="80.137" y="52.6542" size="1.778" layer="95"/>
+<attribute name="VALUE" x="80.137" y="47.498" size="1.778" layer="96"/>
+</instance>
+<instance part="RXARD" gate="1" x="63.5" y="2.54" smashed="yes">
+<attribute name="NAME" x="62.357" y="4.3942" size="1.778" layer="95"/>
+<attribute name="VALUE" x="62.357" y="-0.762" size="1.778" layer="96"/>
+</instance>
+<instance part="TXARD" gate="1" x="63.5" y="5.08" smashed="yes">
+<attribute name="NAME" x="62.357" y="6.9342" size="1.778" layer="95"/>
+<attribute name="VALUE" x="62.357" y="1.778" size="1.778" layer="96"/>
 </instance>
 </instances>
@@
 </busses>
 <nets>
-<net name="N$1" class="0">
-<segment>
-<pinref part="U1" gate="G$1" pin="SCL"/>
-<pinref part="U$1" gate="G$1" pin="A5"/>
-<wire x1="99.06" y1="50.8" x2="45.72" y2="50.8" width="0.1524" layer="91"/>
-<wire x1="45.72" y1="50.8" x2="45.72" y2="43.18" width="0.1524" layer="91"/>
-</segment>
-</net>
-<net name="N$2" class="0">
-<segment>
-<pinref part="U1" gate="G$1" pin="SDA"/>
-<pinref part="U$1" gate="G$1" pin="A4"/>
-<wire x1="99.06" y1="45.72" x2="48.26" y2="45.72" width="0.1524" layer="91"/>
-<wire x1="48.26" y1="45.72" x2="48.26" y2="43.18" width="0.1524" layer="91"/>
-</segment>
-</net>
 <net name="N$4" class="0">
 <segment>
@@
 <wire x1="45.72" y1="71.12" x2="45.72" y2="66.04" width="0.1524" layer="91"/>
 <junction x="45.72" y="71.12"/>
-<pinref part="U$1" gate="G$1" pin="GND"/>
 <wire x1="45.72" y1="66.04" x2="40.64" y2="66.04" width="0.1524" layer="91"/>
-<wire x1="40.64" y1="60.96" x2="40.64" y2="66.04" width="0.1524" layer="91"/>
 <wire x1="40.64" y1="66.04" x2="17.78" y2="66.04" width="0.1524" layer="91"/>
 <pinref part="U$2" gate="G$1" pin="GND"/>
 <wire x1="17.78" y1="66.04" x2="17.78" y2="0" width="0.1524" layer="91"/>
 <wire x1="17.78" y1="0" x2="76.2" y2="0" width="0.1524" layer="91"/>
+<junction x="40.64" y="66.04"/>
+<pinref part="GNDARD" gate="1" pin="P"/>
+<wire x1="40.64" y1="66.04" x2="40.64" y2="45.72" width="0.1524" layer="91"/>
 </segment>
 </net>
 <net name="N$5" class="0">
 <segment>
-<pinref part="U$1" gate="G$1" pin="TX0"/>
 <pinref part="U$2" gate="G$1" pin="RX"/>
-<wire x1="38.1" y1="17.78" x2="38.1" y2="5.08" width="0.1524" layer="91"/>
-<wire x1="38.1" y1="5.08" x2="76.2" y2="5.08" width="0.1524" layer="91"/>
+<wire x1="66.04" y1="5.08" x2="76.2" y2="5.08" width="0.1524" layer="91"/>
+<pinref part="TXARD" gate="1" pin="P"/>
 </segment>
 </net>
 <net name="N$6" class="0">
 <segment>
-<pinref part="U$1" gate="G$1" pin="RX1"/>
 <pinref part="U$2" gate="G$1" pin="TX"/>
-<wire x1="40.64" y1="17.78" x2="40.64" y2="2.54" width="0.1524" layer="91"/>
-<wire x1="40.64" y1="2.54" x2="76.2" y2="2.54" width="0.1524" layer="91"/>
+<wire x1="66.04" y1="2.54" x2="76.2" y2="2.54" width="0.1524" layer="91"/>
+<pinref part="RXARD" gate="1" pin="P"/>
 </segment>
 </net>
@@
 <wire x1="66.04" y1="78.74" x2="78.74" y2="78.74" width="0.1524" layer="91"/>
 <wire x1="78.74" y1="78.74" x2="99.06" y2="78.74" width="0.1524" layer="91"/>
-<pinref part="U$1" gate="G$1" pin="RAW"/>
-<wire x1="38.1" y1="88.9" x2="38.1" y2="73.66" width="0.1524" layer="91"/>
-<wire x1="38.1" y1="73.66" x2="38.1" y2="60.96" width="0.1524" layer="91"/>
+<wire x1="38.1" y1="88.9" x2="38.1" y2="78.74" width="0.1524" layer="91"/>
+<wire x1="38.1" y1="78.74" x2="38.1" y2="73.66" width="0.1524" layer="91"/>
 <wire x1="38.1" y1="73.66" x2="15.24" y2="73.66" width="0.1524" layer="91"/>
-<junction x="38.1" y="73.66"/>
 <pinref part="U$2" gate="G$1" pin="+5V"/>
 <wire x1="15.24" y1="73.66" x2="15.24" y2="-2.54" width="0.1524" layer="91"/>
-<wire x1="15.24" y1="-2.54" x2="63.5" y2="-2.54" width="0.1524" layer="91"/>
-<pinref part="U$2" gate="G$1" pin="EN"/>
-<wire x1="63.5" y1="-2.54" x2="76.2" y2="-2.54" width="0.1524" layer="91"/>
-<wire x1="63.5" y1="-2.54" x2="63.5" y2="-5.08" width="0.1524" layer="91"/>
-<wire x1="63.5" y1="-5.08" x2="76.2" y2="-5.08" width="0.1524" layer="91"/>
-<junction x="63.5" y="-2.54"/>
+<wire x1="15.24" y1="-2.54" x2="76.2" y2="-2.54" width="0.1524" layer="91"/>
 <wire x1="78.74" y1="78.74" x2="78.74" y2="88.9" width="0.1524" layer="91"/>
 <wire x1="78.74" y1="88.9" x2="38.1" y2="88.9" width="0.1524" layer="91"/>
 <junction x="78.74" y="78.74"/>
+<pinref part="VCCARD" gate="1" pin="P"/>
+<wire x1="22.86" y1="78.74" x2="38.1" y2="78.74" width="0.1524" layer="91"/>
+<junction x="38.1" y="78.74"/>
 </segment>
 </net>
@@
 <pinref part="VCC" gate="1" pin="P"/>
 <pinref part="INTER1" gate="1" pin="P"/>
-<wire x1="45.72" y1="78.74" x2="55.88" y2="78.74" width="0.1524" layer="91"/>
+<wire x1="48.26" y1="78.74" x2="55.88" y2="78.74" width="0.1524" layer="91"/>
+</segment>
+</net>
+<net name="N$1" class="0">
+<segment>
+<pinref part="A5ARD" gate="1" pin="P"/>
+<pinref part="U1" gate="G$1" pin="SCL"/>
+<wire x1="83.82" y1="50.8" x2="99.06" y2="50.8" width="0.1524" layer="91"/>
+</segment>
+</net>
+<net name="N$2" class="0">
+<segment>
+<pinref part="A4ARD" gate="1" pin="P"/>
+<pinref part="U1" gate="G$1" pin="SDA"/>
+<wire x1="83.82" y1="45.72" x2="99.06" y2="45.72" width="0.1524" layer="91"/>
 </segment>
 </net>
@@
 </schematic>
 </drawing>
-<compatibility>
-<note version="8.2" severity="warning">
-Since Version 8.2, EAGLE supports online libraries. The ids
-of those online libraries will not be understood (or retained)
-with this version.
-</note>
-<note version="8.3" severity="warning">
-Since Version 8.3, EAGLE supports URNs for individual library
-assets (packages, symbols, and devices). The URNs of those assets
-will not be understood (or retained) with this version.
-</note>
-<note version="8.3" severity="warning">
-Since Version 8.3, EAGLE supports the association of 3D packages
-with devices in libraries, schematics, and board files. Those 3D
-packages will not be understood (or retained) with this version.
-</note>
-</compatibility>
 </eagle>
